Commit message: [fallschool] adding new pr2 config for costmap show in rviz web

File: resources/apartment-small.urdf (robot description, URDF)
Before this commit: robot apartment, 102 links, 101 joints
Links:
- removed link bedside_table
- removed link coffee_table
- removed link coffee_table_drawer
- removed link sofa
Joints:
- removed joint bedside_table_joint
- removed joint coffee_table_drawer_joint
- removed joint coffee_table_joint
- removed joint sofa_joint
