Commit message: [vib] added floor

File: resources/objects/plane_colored.urdf (robot description, URDF)
Before this commit: robot plane, 1 links, 0 joints
Links:
- link planeLink: geometry collision mesh filename=package://pycram/resources/plane.obj scale=0.64 0.17 0.4; visual mesh filename=plane.obj scale=0.64 0.17 0.4
